File: redbearpad.kicad_pcb (KiCad board)
At the start: 2 copper layers, 96 x 64 mm, 15 parts, among them J1 PinSocket_1x14_P2.54mm_Vertic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, J2 PinSocket_1x14_P2.54mm_Vertic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, J3 PinSocket_1x04_P2.54mm_Vertic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, SW1 SW_Redragon_LowProfile_PCB_1.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, SW2 SW_Redragon_LowProfile_PCB_1.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, SW3 SW_Redragon_LowProfile_PCB_1.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, SW4 SW_Redragon_LowProfile_PCB_1.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, SW5 SW_Redragon_LowProfile_PCB_1.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, SW6 SW_Redragon_LowProfile_PCB_1.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, SW7 SW_Redragon_LowProfile_PCB_1.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, SW8 SW_Redragon_LowProfile_PCB_1.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

Commit message: Ruteo final: DRC sin errores ni unconnected
Co-Authored-By: Claude Fable 5 <noreply@anthropic.com>
Routing:
- net SW8: track 45.4 -> 66.6 mm
- net SW4: track 31.2 -> 43.5 mm
- net SW6: track 15.6 -> 24.7 mm
- net SW7: track 33.2 -> 42.0 mm
- net SW3: track 68.0 -> 59.6 mm
- net +3V3: track 91.7 -> 99.7 mm
- net SW5: track 27.1 -> 24.1 mm
- net SW1: track 25.1 -> 24.5 mm
