File: redbearpad.kicad_pcb (KiCad board)
At the start: 2 copper layers, 96 x 64 mm, 18 parts, among them J1 PinSocket_1x14_P2.54mm_Vertic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, J2 PinSocket_1x14_P2.54mm_Vertic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, SW1 SW_Redragon_LowProfile_PCB_1.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, SW10 SW_Redragon_LowProfile_PCB_1.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, SW11 SW_Tact_CAX, SW12 SW_Tact_CAX, SW2 SW_Redragon_LowProfile_PCB_1.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, SW3 SW_Redragon_LowProfile_PCB_1.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, SW4 SW_Redragon_LowProfile_PCB_1.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, SW5 SW_Redragon_LowProfile_PCB_1.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, SW6 SW_Redragon_LowProfile_PCB_1.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, SW7 SW_Redragon_LowProfile_PCB_1.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, SW8 SW_Redragon_LowProfile_PCB_1.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, SW9 SW_Redragon_LowProfile_PCB_1.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

Commit message: feat(3d): placeholder dimensionalmente real de la Blend Micro
Se descarta usar un modelo de Arduino Micro como sustituto: sus medidas
oficiales (48x18mm) no calzan con la Blend Micro real (42.087x18.4mm,
confirmado contra el DXF oficial del fabricante) -- 14% mas larga, y
probablemente con headers en otro patron. Sustituirlo habria dado un
render dimensionalmente falso.

En su lugar se genera un placeholder propio a partir de datos reales:

- scripts/gen_blendmicro_step.py: extruye con CadQuery una placa plana
  18.4x42.087mm, esquinas R=1.42mm. Ancho/largo/radio de esquina salen
  del contorno real en blend-micro-boards/upstream/Blend/PCB/
  Blend_Micro.dxf (capa BOARD_OUTLINE_00, geometria dentro de un bloque
  BOARD_36 -- hubo que aplicar la transformacion del INSERT via
  ezdxf.virtual_entities() para sacar coordenadas de mundo). El radio de
  esquina se calculo desde el bulge de la LWPOLYLINE (bulge=-0.4132 ->
  angulo ~90 grados -> R=1.42mm). Grosor 1.6mm: ESTANDAR ASUMIDO, el DXF
  es 2D y no lo especifica.
- libs/redbearpad.pretty/BlendMicro_Module.kicad_mod: footprint SIN pads
  (la conexion real la hacen J1/J2); solo courtyard/fab + el modelo 3D.
  Se quito el B.CrtYd que se probo primero: el modulo se enchufa DENTRO
  de J1/J2 por diseno, asi que su courtyard SIEMPRE va a solapar el de
  los zocalos -- no es un error de colocacion, es dos DRC courtyards
  overlap esperables que se evitan no dandole courtyard a un footprint
  no-electrico.
- scripts/insert_blendmicro_footprint.py: inserta BLENDMICRO1 en (48.0,
  21.044) -- centro X entre J1/J2, Y tal que el borde superior del
  modulo caiga en y=0 (coincide con el borde superior de la placa, tal
  como documenta el spec original). Sin regenerar el board (no pierde
  ruteo), igual que attach_3d_models.py.
- scripts/gen_pcb.py: se agrega BLENDMICRO1 al dict PLACE para que una
  regeneracion completa futura ya lo traiga.

Verificado: netlist OK, DRC de cobre limpio (0 sin conectar, las 8
avisos cosmeticas de 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
Parts:
- added BLENDMICRO1: BlendMicro_Module, BlendMicro_Module, B.Cu at (48.0, 21.0)
Changed lines of the file:
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@@
 		(embedded_fonts no)
+	)
+	(footprint "BlendMicro_Module"
+		(layer "B.Cu")
+		(at 48 21.044)
+		(descr "Representacion visual (sin pads) del modulo RedBearLab Blend Micro V1.0 enchufado en J1/J2. Medidas reales del DXF oficial del fabricante: 18.4x42.087mm. No lleva conexion electrica: la conectan J1/J2.")
+		(tags "RedBearLab Blend Micro visual placeholder no-connect")
+		(property "Reference" "BLENDMICRO1"
+			(at 0 -23.5 0)
+			(layer "B.SilkS")
+			(effects
+				(font
+					(size 1 1)
+					(thickness 0.15)
+				)
+				(justify mirror)
+			)
+		)
+		(property "Value" "BlendMicro_Module"
+			(at 0 23.5 0)
+			(layer "B.Fab")
+			(effects
+				(font
+					(size 1 1)
+					(thickness 0.15)
+				)
+				(justify mirror)
+			)
+		)
+		(property "Datasheet" ""
+			(at 0 0 0)
+			(layer "F.Fab")
+			(hide yes)
+			(effects
+				(font
+					(size 1.27 1.27)
+					(thickness 0.15)
+				)
+			)
+		)
+		(property "Description" ""
+			(at 0 0 0)
+			(layer "F.Fab")
+			(hide yes)
+			(effects
+				(font
+					(size 1.27 1.27)
+					(thickness 0.15)
+				)
+			)
+		)
+		(attr exclude_from_pos_files exclude_from_bom allow_missing_courtyard)
+		(fp_rect
+			(start -9.2 -21.044)
+			(end 9.2 21.044)
+			(stroke
+				(width 0.1)
+				(type solid)
+			)
+			(fill no)
+			(layer "B.Fab")
+		)
+		(embedded_fonts no)
+		(model "${KIPRJMOD}/libs/redbearpad.3dshapes/BlendMicro_Module.step"
+			(offset
+				(xyz 0 0 0)
+			)
+			(scale
+				(xyz 1 1 1)
+			)
+			(rotate
+				(xyz 0 0 0)
+			)
+		)
 	)
 	(footprint "PinSocket_1x14_P2.54mm_Vertical"
